File: Digital Potentiometer Module.kicad_sch (KiCad schematic)
At the start: 17 parts, among them J1 Barrel_Jack, J2 Conn_01x04_Pin, J3 Conn_01x02_Pin, SW1 SW_SPST, SW2 SW_SPST, U1 ESP32-WROOM-32E, U2 AD5231BRUZ10, U3 LM317_SOT-223

Commit message: add footprints
Parts:
- C1, C2: value C_Polarized -> 10uF; footprint (none) -> Capacitor_SMD:CP_Elec_5x5.3
- D1: footprint (none) -> LED_SMD:LED_0603_1608Metric_Pad1.05x0.95mm_HandSolder
- J1: value Barrel_Jack -> Barrel_Jack (>5V)
- J2: footprint (none) -> Connector_PinHeader_2.54mm:PinHeader_1x04_P2.54mm_Vertical
- J3: footprint (none) -> Connector_PinHeader_2.54mm:PinHeader_1x02_P2.54mm_Vertical
- R1, R2, R3, R4, R5: footprint (none) -> Resistor_SMD:R_0805_2012Metric_Pad1.20x1.40mm_HandSolder
- SW1, SW2: footprint (none) -> Button_Switch_SMD:SW_SPST_PTS645
- renumbered D1 to D2
Connections:
- net 3.3V: now also R3.1; no longer R3.2
- net GND: now also R5.1, U3.1 (ADJ); no longer R5.2
- net at SW1.1 (A), U1.3 (EN): now also R3.2; no longer R3.1
- new net: R4.2, R5.2
Other:
- moved on the sheet: R3, R5
Changed lines of the file:
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@@
 	)
 	(junction
-		(at 245.11 115.57)
+		(at 67.31 40.64)
 		(diameter 0)
 		(color 0 0 0 0)
@@
 	)
 	(junction
-		(at 78.74 49.53)
+		(at 78.74 30.48)
 		(diameter 0)
 		(color 0 0 0 0)
 	)
 	(junction
-		(at 78.74 30.48)
+		(at 246.38 115.57)
 		(diameter 0)
 		(color 0 0 0 0)
@@
 	)
 	(junction
-		(at 78.74 40.64)
-		(diameter 0)
-		(color 0 0 0 0)
-	)
-	(junction
 		(at 67.31 49.53)
 		(diameter 0)
@@
 	(wire
 		(pts
-			(xy 245.11 115.57) (xy 245.11 118.11)
-		)
-		(stroke
-			(width 0)
-			(type default)
-		)
-	)
-	(wire
-		(pts
 			(xy 57.15 35.56) (xy 57.15 49.53)
 		)
@@
 	(wire
 		(pts
+			(xy 246.38 115.57) (xy 246.38 121.92)
+		)
+		(stroke
+			(width 0)
+			(type default)
+		)
+	)
+	(wire
+		(pts
 			(xy 55.88 30.48) (xy 59.69 30.48)
 		)
@@
 	(wire
 		(pts
-			(xy 228.6 115.57) (xy 245.11 115.57)
-		)
-		(stroke
-			(width 0)
-			(type default)
-		)
-	)
-	(wire
-		(pts
 			(xy 266.065 130.81) (xy 234.95 130.81)
 		)
@@
 	(wire
 		(pts
-			(xy 78.74 49.53) (xy 92.71 49.53)
-		)
-		(stroke
-			(width 0)
-			(type default)
-		)
-	)
-	(wire
-		(pts
 			(xy 191.77 64.77) (xy 198.12 64.77)
 		)
@@
 	(wire
 		(pts
+			(xy 67.31 49.53) (xy 92.71 49.53)
+		)
+		(stroke
+			(width 0)
+			(type default)
+		)
+	)
+	(wire
+		(pts
 			(xy 213.36 38.1) (xy 220.98 38.1)
 		)
@@
 	(wire
 		(pts
-			(xy 78.74 48.26) (xy 78.74 49.53)
-		)
-		(stroke
-			(width 0)
-			(type default)
-		)
-	)
-	(wire
-		(pts
-			(xy 67.31 40.64) (xy 78.74 40.64)
+			(xy 67.31 40.64) (xy 67.31 49.53)
 		)
 		(stroke
@@
 	(wire
 		(pts
+			(xy 246.38 115.57) (xy 252.73 115.57)
+		)
+		(stroke
+			(width 0)
+			(type default)
+		)
+	)
+	(wire
+		(pts
 			(xy 29.21 104.14) (xy 29.21 111.76)
 		)
@@
 	(wire
 		(pts
-			(xy 245.11 115.57) (xy 252.73 115.57)
-		)
-		(stroke
-			(width 0)
-			(type default)
-		)
-	)
-	(wire
-		(pts
-			(xy 67.31 49.53) (xy 78.74 49.53)
+			(xy 228.6 115.57) (xy 246.38 115.57)
+		)
+		(stroke
+			(width 0)
+			(type default)
+		)
+	)
+	(wire
+		(pts
+			(xy 76.2 40.64) (xy 78.74 40.64)
 		)
 		(stroke
@@
 		(pts
 			(xy 29.21 116.84) (xy 29.21 120.65)
+		)
+		(stroke
+			(width 0)
+			(type default)
+		)
+	)
+	(wire
+		(pts
+			(xy 67.31 40.64) (xy 68.58 40.64)
 		)
 		(stroke
@@
 	)
 	(label "3.3V"
-		(at 245.11 125.73 270)
+		(at 238.76 121.92 180)
 		(fields_autoplaced yes)
 		(effects
@@
 			)
 		)
-		(property "Footprint" ""
+		(property "Footprint" "Resistor_SMD:R_0805_2012Metric_Pad1.20x1.40mm_HandSolder"
 			(at 76.962 36.83 90)
 			(effects
@@
 			)
 		)
-		(property "Footprint" ""
+		(property "Footprint" "Button_Switch_SMD:SW_SPST_PTS645"
 			(at 257.81 115.57 0)
 			(effects
@@
 			)
 		)
-		(property "Footprint" ""
+		(property "Footprint" "Button_Switch_SMD:SW_SPST_PTS645"
 			(at 179.07 115.57 0)
 			(effects
@@
 	(symbol
 		(lib_id "Device:R")
-		(at 245.11 121.92 0)
+		(at 242.57 121.92 90)
 		(unit 1)
 		(exclude_from_sim no)
@@
 		(fields_autoplaced yes)
 		(property "Reference" "R3"
-			(at 247.65 120.6499 0)
-			(effects
-				(font
-					(size 1.27 1.27)
-				)
-				(justify left)
+			(at 242.57 115.57 90)
+			(effects
+				(font
+					(size 1.27 1.27)
+				)
 			)
 		)
 		(property "Value" "10K"
-			(at 247.65 123.1899 0)
-			(effects
-				(font
-					(size 1.27 1.27)
-				)
-				(justify left)
-			)
-		)
-		(property "Footprint" ""
-			(at 243.332 121.92 90)
+			(at 242.57 118.11 90)
+			(effects
+				(font
+					(size 1.27 1.27)
+				)
+			)
+		)
+		(property "Footprint" "Resistor_SMD:R_0805_2012Metric_Pad1.20x1.40mm_HandSolder"
+			(at 242.57 123.698 90)
 			(effects
 				(font
@@
 		)
 		(property "Datasheet" "~"
-			(at 245.11 121.92 0)
+			(at 242.57 121.92 0)
 			(effects
 				(font
@@
 		)
 		(property "Description" "Resistor"
-			(at 245.11 121.92 0)
+			(at 242.57 121.92 0)
 			(effects
 				(font
@@
 			)
 		)
-		(property "Footprint" ""
+		(property "Footprint" "Resistor_SMD:R_0805_2012Metric_Pad1.20x1.40mm_HandSolder"
 			(at 90.932 34.29 90)
 			(effects
@@
 			)
 		)
-		(property "Footprint" ""
+		(property "Footprint" "Connector_PinHeader_2.54mm:PinHeader_1x02_P2.54mm_Vertical"
 			(at 64.77 148.59 0)
 			(effects
@@
 			)
 		)
-		(property "Footprint" ""
+		(property "Footprint" "Resistor_SMD:R_0805_2012Metric_Pad1.20x1.40mm_HandSolder"
 			(at 189.992 124.46 90)
 			(effects
@@
 	(symbol
 		(lib_id "Device:R")
-		(at 78.74 44.45 0)
+		(at 72.39 40.64 90)
 		(unit 1)
 		(exclude_from_sim no)
@@
 		(fields_autoplaced yes)
 		(property "Reference" "R5"
-			(at 81.28 43.1799 0)
-			(effects
-				(font
-					(size 1.27 1.27)
-				)
-				(justify left)
+			(at 72.39 34.29 90)
+			(effects
+				(font
+					(size 1.27 1.27)
+				)
 			)
 		)
 		(property "Value" "360"
-			(at 81.28 45.7199 0)
-			(effects
-				(font
-					(size 1.27 1.27)
-				)
-				(justify left)
-			)
-		)
-		(property "Footprint" ""
-			(at 76.962 44.45 90)
+			(at 72.39 36.83 90)
+			(effects
+				(font
+					(size 1.27 1.27)
+				)
+			)
+		)
+		(property "Footprint" "Resistor_SMD:R_0805_2012Metric_Pad1.20x1.40mm_HandSolder"
+			(at 72.39 42.418 90)
 			(effects
 				(font
@@
 		)
 		(property "Datasheet" "~"
-			(at 78.74 44.45 0)
+			(at 72.39 40.64 0)
 			(effects
 				(font
@@
 		)
 		(property "Description" "Resistor"
-			(at 78.74 44.45 0)
+			(at 72.39 40.64 0)
 			(effects
 				(font
@@
 			)
 		)
-		(property "Value" "C_Polarized"
+		(property "Value" "10uF"
 			(at 226.441 125.73 90)
 			(effects
@@
 			)
 		)
-		(property "Footprint" ""
+		(property "Footprint" "Capacitor_SMD:CP_Elec_5x5.3"
 			(at 231.14 129.8448 0)
 			(effects
@@
 			)
 		)
-		(property "Footprint" ""
+		(property "Footprint" "LED_SMD:LED_0603_1608Metric_Pad1.05x0.95mm_HandSolder"
 			(at 92.71 45.72 0)
 			(effects
@@
 			)
 		)
-		(property "Value" "Barrel_Jack"
+		(property "Value" "Barrel_Jack (>5V)"
 			(at 30.48 26.67 0)
 			(effects
@@
 			)
 		)
-		(property "Value" "C_Polarized"
+		(property "Value" "10uF"
 			(at 225.679 33.02 90)
 			(effects
@@
 			)
 		)
-		(property "Footprint" ""
+		(property "Footprint" "Capacitor_SMD:CP_Elec_5x5.3"
 			(at 220.98 39.0652 0)
 			(effects
@@
 				)
 				(hide yes)
+			)
+		)
+		(property "Purpose" ""
+			(at 224.79 38.1 0)
+			(effects
+				(font
+					(size 1.27 1.27)
+				)
 			)
 		)
@@
 			)
 		)
-		(property "Footprint" ""
+		(property "Footprint" "Connector_PinHeader_2.54mm:PinHeader_1x04_P2.54mm_Vertical"
 			(at 38.1 152.4 0)
 			(effects
@@
 		(dnp no)
 		(fields_autoplaced yes)
-		(property "Reference" "D1"
+		(property "Reference" "D2"
 			(at 52.07 24.13 0)
 			(effects
@@
 			(project "Digital Potentiometer Module"
 				(path "/f9605a72-0ec6-49c8-8d90-8c2a65c3e011"
-					(reference "D1")
+					(reference "D2")
 					(unit 1)
 				)
