File: Digital Potentiometer Module.kicad_sch (KiCad schematic)
At the start: 18 parts, among them J1 Barrel_Jack (>5V), J2 Conn_01x04_Pin, J3 Conn_01x02_Pin, J4 Conn_01x03_Pin, SW1 SW_SPST, SW2 SW_SPST, U1 ESP32-WROOM-32E, U2 AD5231BRUZ10, U3 LM317_SOT-223

Commit message: make improvements to pcb
Parts:
- removed J3: Conn_01x02_Pin, Connector_PinHeader_2.54mm:PinHeader_1x02_P2.54mm_Vertical, symbol Connector:Conn_01x02_Pin
- added J5: Conn_01x03_Pin, Connector_PinHeader_2.54mm:PinHeader_1x03_P2.54mm_Vertical, symbol Connector:Conn_01x03_Pin
- added S1: Slide Switch, digikey-footprints:Switch_Slide_11.6x4mm_EG1218, symbol dk_Slide-Switches:EG1218
- U1: footprint RF_Module:ESP32-WROOM-32D -> Custom:XCVR_ESP32-WROOM-32E__4MB_
Connections:
- net 3.3V: now also S1.3
- net ENC_A: now also J5.1 (Pin_1)
- net ENC_B: now also J5.3 (Pin_3)
- net GND: now also J5.2 (Pin_2)
- net VIN: now also S1.1; no longer D2.1 (K)
- net BOOT: now reaches R1.1, SW2.2 (B), U1.25 (IO0)
- net EN: now reaches R3.2, SW1.1 (A), U1.3 (EN)
- net J_POS renamed PD_IN
- new net PD_OUT: D2.1 (K), S1.2
Other:
- moved on the sheet: D1, J1, R2, R4, R5, U3
