File: _autosave-Digital Potentiometer Module.kicad_sch (KiCad schematic)
At the start: 18 parts, among them J1 Barrel_Jack (>5V), J2 Conn_01x04_Pin, J3 Conn_01x02_Pin, J4 Conn_01x03_Pin, SW1 SW_SPST, SW2 SW_SPST, U1 ESP32-WROOM-32E, U2 AD5231BRUZ10, U3 LM317_SOT-223

Commit message: design pcb
Parts:
- added S1: Slide Switch, digikey-footprints:Switch_Slide_11.6x4mm_EG1218, symbol dk_Slide-Switches:EG1218
Connections:
- net 3.3V: now also S1.3
- net VIN: now also S1.1; no longer D2.1 (K)
- net BOOT: now reaches R1.1, SW2.2 (B), U1.25 (IO0)
- net EN: now reaches R3.2, SW1.1 (A), U1.3 (EN)
- new net: D2.1 (K), S1.2
Other:
- moved on the sheet: D1, D2, J1, R2, R4, R5, U3
